Commit message: Manual and rviz working

File: rocky/src/rocky_description/urdf/lidar.xacro (robot description, xacro)
@@ -4,5 +4,5 @@
         <parent link="chassis"/>
         <child link="laser_frame"/>
-        <origin xyz="0.122 0 0.05" rpy="0 0 0"/>
+        <origin xyz="0.122 0 0.212" rpy="0 0 0"/>
     </joint>
     <link name="laser_frame">
@@ -31,5 +31,5 @@
  <gazebo reference="laser_frame">
     <material>Gazebo/Black</material>
-    <sensor name="laser" type="lidar">
+    <sensor name="laser" type="gpu_lidar">
         <always_on>true</always_on>
         <visualize>true</visualize>
