Commit message: multiple changes, manual working , autonomous not yet

File: rocky/src/rocky_description/urdf/camera.xacro (robot description, xacro)
@@ -11,5 +11,5 @@
                 <box size="0.010 0.03 0.03"/>
             </geometry>
-            <material name="red"/>
+            <material name="rocky_red"/>
         </visual>
     </link>
@@ -38,7 +38,11 @@
                 </clip>
             </camera>
-            <plugin name="camera_controller" filename="libgazebo_ros_camera.so">
+            <!-- <plugin name="camera_controller" filename="libgazebo_ros_camera.so">
                 <frame_name>camera_link_optical</frame_name>
-            </plugin>
+            </plugin> -->
+            <!-- <plugin filename="gz-sim-sensors-system" name="gz::sim::systems::Sensors">
+            <render_engine>ogre2</render_engine>
+            </plugin> -->
+<!-- topic is set via <topic> tag on the <sensor> element -->
         </sensor>
     </gazebo>

File: rocky/src/rocky_description/urdf/depth_camera.xacro (robot description, xacro)
@@ -11,5 +11,5 @@
                 <box size="0.010 0.03 0.03"/>
             </geometry>
-            <material name="red"/>
+            <material name="rocky_red"/>
         </visual>
     </link>
@@ -38,9 +38,15 @@
                 </clip>
             </camera>
-            <plugin name="camera_controller" filename="libgazebo_ros_camera.so">
+            <!-- <plugin name="camera_controller" filename="libgazebo_ros_camera.so">
                 <frame_name>camera_link_optical</frame_name>
                 <min_depth>0.1</min_depth>
                 <max_depth>8.0</max_depth>
-             </plugin>
+             </plugin> -->
+             <!-- <plugin filename="gz-sim-sensors-system" name="gz::sim::systems::Sensors">
+            <render_engine>ogre2</render_engine>
+            <min_depth>0.1</min_depth>
+                <max_depth>8.0</max_depth>
+            </plugin> -->
+<!-- topic is set via <topic> tag on the <sensor> element -->
         </sensor>
     </gazebo>

File: rocky/src/rocky_description/urdf/gazebo_control.xacro (robot description, xacro)
@@ -2,5 +2,6 @@
 <robot xmlns:xacro="http://www.ros.org/wiki/xacro">
     <gazebo>
-        <plugin name="diff_drive" filename="libgazebo_ros_diff_drive.so">
+        <!-- <plugin name="diff_drive" filename="libgazebo_ros_diff_drive.so"> -->
+        <plugin filename="gz-sim-diff-drive-system" name="gz::sim::systems::DiffDrive">
             <!-- Wheel Information -->
             <left_joint>left_wheel_joint</left_joint>

File: rocky/src/rocky_description/urdf/imu.xacro (robot description, xacro)
@@ -11,5 +11,5 @@
                 <box size="0.02 0.02 0.02"/>
             </geometry>
-            <material name="black"/>
+            <material name="rocky_black"/>
         </visual>
     </link>
@@ -20,4 +20,6 @@
             <update_rate>100</update_rate>
             <visualize>true</visualize>
+            <topic>imu</topic>
+            <gz_frame_id>imu_link</gz_frame_id>
             <imu>
                 <angular_velocity>
@@ -62,10 +64,12 @@
                 </linear_acceleration>
             </imu>
-            <plugin filename="libgazebo_ros_imu_sensor.so" name="imu_plugin">
+            <!-- <plugin filename="libgazebo_ros_imu_sensor.so" name="imu_plugin">
                 <ros>
                     <remapping>~/out:=imu</remapping>
                 </ros>
                 <initial_orientation_as_reference>false</initial_orientation_as_reference>
-            </plugin>
+            </plugin> -->
+            <plugin filename="gz-sim-imu-system"
+            name="gz::sim::systems::Imu"/>
         </sensor>
     </gazebo>

File: rocky/src/rocky_description/urdf/lidar.xacro (robot description, xacro)
@@ -4,5 +4,5 @@
         <parent link="chassis"/>
         <child link="laser_frame"/>
-        <origin xyz="0.122 0 0.212" rpy="0 0 0"/>
+        <origin xyz="0.122 0 0.05" rpy="0 0 0"/>
     </joint>
     <link name="laser_frame">
@@ -11,5 +11,5 @@
                 <cylinder radius="0.05" length="0.04"/>
             </geometry>
-            <material name="black"/>
+            <material name="rocky_black"/>
         </visual>
         <visual>
@@ -18,5 +18,5 @@
                 <cylinder radius="0.01" length="0.1"/>
             </geometry>
-            <material name="black"/>
+            <material name="rocky_black"/>
         </visual>
         <collision>
@@ -29,32 +29,33 @@
         </xacro:inertial_cylinder>
     </link>
-    <gazebo reference="laser_frame">
-        <material>Gazebo/Black</material>
-        <sensor name="laser" type="gpu_ray">
-            <pose> 0 0 0 0 0 0 </pose>
-            <visualize>true</visualize> <update_rate>10</update_rate>
-            <ray>
-                <scan>
-                    <horizontal>
-                        <samples>360</samples>
-                        <resolution>1</resolution>
-                        <min_angle>-3.14159</min_angle>
-                        <max_angle>3.14159</max_angle>
-                    </horizontal>
-                    </scan>
-                <range>
-                    <min>0.1</min>
-                    <max>12.0</max>
-                    <resolution>0.01</resolution>
-                </range>
-            </ray>
-            <plugin name="laser_controller" filename="libgazebo_ros_ray_sensor.so">
-                <ros>
-                    <argument>~/out:=scan</argument>
-                </ros>
-                <output_type>sensor_msgs/LaserScan</output_type>
-                <frame_name>laser_frame</frame_name>
-            </plugin>
-        </sensor>
-    </gazebo>
+ <gazebo reference="laser_frame">
+    <material>Gazebo/Black</material>
+    <sensor name="laser" type="lidar">
+        <always_on>true</always_on>
+        <visualize>true</visualize>
+        <update_rate>10</update_rate>
+        <topic>scan</topic>
+        <gz_frame_id>laser_frame</gz_frame_id>
+        <ray>
+            <scan>
+                <horizontal>
+                    <samples>360</samples>
+                    <resolution>1.0</resolution>
+                    <min_angle>-3.14159</min_angle>
+                    <max_angle>3.14159</max_angle>
+                </horizontal>
+            </scan>
+            <range>
+                <min>0.1</min>
+                <max>12.0</max>
+                <resolution>0.015</resolution>
+            </range>
+            <noise>
+                <type>gaussian</type>
+                <mean>0.0</mean>
+                <stddev>0.01</stddev>
+            </noise>
+        </ray>
+    </sensor>
+</gazebo>
 </robot>

File: rocky/src/rocky_description/urdf/rocky_core.xacro (robot description, xacro)
@@ -16,17 +16,17 @@
     <xacro:property name="caster_wheel_offset_x" value="0.075"/>
     <xacro:property name="caster_wheel_offset_z" value="${wheel_offset_z - wheel_radius + caster_wheel_radius}"/>
-    <material name="white">
+    <material name="rocky_white">
         <color rgba="1 1 1 1" />
     </material>
-    <material name="orange">
+    <material name="rocky_orange">
         <color rgba="1 0.3 0.1 1"/>
     </material>
-    <material name="blue">
+    <material name="rocky_blue">
         <color rgba="0.2 0.2 1 1"/>
     </material>
-    <material name="black">
+    <material name="rocky_black">
         <color rgba="0 0 0 1"/>
     </material>
-    <material name="red">
+    <material name="rocky_red">
         <color rgba="1 0 0 1"/>
     </material>
@@ -35,9 +35,14 @@
     </link>
     <!-- BASE_FOOTPRINT LINK -->
-    <joint name="base_footprint_joint" type="fixed">
+    <!-- <joint name="base_footprint_joint" type="fixed">
             <parent link="base_footprint"/>
             <child link="base_link"/>
             <origin xyz="0 0 0" rpy="0 0 0"/>
-        </joint>
+        </joint> -->
+<joint name="base_footprint_joint" type="fixed">
+        <parent link="base_footprint"/>
+        <child link="base_link"/>
+        <origin xyz="0 0 0.033" rpy="0 0 0"/>
+    </joint>
     <link name="base_footprint">
     </link>
@@ -54,5 +59,5 @@
                 <box size="${chassis_length} ${chassis_width} ${chassis_height}"/>
             </geometry>
-            <material name="orange"/>
+            <material name="rocky_orange"/>
         </visual>
         <collision>
@@ -81,9 +86,9 @@
                 <cylinder radius="${wheel_radius}" length="${wheel_thickness}"/>
             </geometry>
-            <material name="blue"/>
+            <material name="rocky_blue"/>
         </visual>
         <collision>
             <geometry>
-                <sphere radius="${wheel_radius}"/>
+                <cylinder radius="${wheel_radius}" length="${wheel_thickness}"/>
             </geometry>
         </collision>
@@ -94,4 +99,6 @@
     <gazebo reference="left_wheel">
         <material>Gazebo/Blue</material>
+     <mu1>1.0</mu1>
+<mu2>1.0</mu2>
     </gazebo>
     <!-- RIGHT WHEEL LINK -->
@@ -107,9 +114,9 @@
                 <cylinder radius="${wheel_radius}" length="${wheel_thickness}"/>
             </geometry>
-            <material name="blue"/>
+            <material name="rocky_blue"/>
         </visual>
         <collision>
             <geometry>
-                <sphere radius="${wheel_radius}"/>
+                <sphere radius="${wheel_radius}" length="${wheel_thickness}"/>
             </geometry>
         </collision>
@@ -120,4 +127,6 @@
     <gazebo reference="right_wheel">
         <material>Gazebo/Blue</material>
+       <mu1>1.0</mu1>
+<mu2>1.0</mu2>
     </gazebo>
     <!-- CASTER WHEEL LINK -->
@@ -132,9 +141,9 @@
                 <sphere radius="${caster_wheel_radius}"/>
             </geometry>
-            <material name="white"/>
+            <material name="rocky_white"/>
         </visual>
         <collision>
             <geometry>
-                <sphere radius="${caster_wheel_radius}"/>
+                <sphere radius="${caster_wheel_radius}" value="0.015"/>
             </geometry>
         </collision>
@@ -143,8 +152,8 @@
         </xacro:inertial_sphere>
     </link>
-    <gazebo reference="caster_wheel">
+  <gazebo reference="caster_wheel">
         <material>Gazebo/White</material>
-        <mu1 value="0.001"/>
-        <mu2 value="0.001"/>
+        <mu1>0.00001</mu1>
+        <mu2>0.00001</mu2>
     </gazebo>
 </robot>

File: rocky/src/rocky_description/urdf/ros2_control.xacro (robot description, xacro)
@@ -34,5 +34,6 @@
         <ros2_control name="GazeboSystem" type="system">
             <hardware>
-                <plugin>gazebo_ros2_control/GazeboSystem</plugin>
+                <!-- <plugin>gazebo_ros2_control/GazeboSystem</plugin> -->
+                <plugin>gz_ros2_control/GazeboSimSystem</plugin>
             </hardware>
             <joint name="left_wheel_joint">
@@ -54,9 +55,15 @@
         </ros2_control>
     </xacro:if>
-    <gazebo>
+    <!-- <gazebo>
         <plugin name="gazebo_ros2_control" filename="libgazebo_ros2_control.so">
             <parameters>$(find rocky_controller)/config/my_controllers.yaml</parameters>
             <parameters>$(find rocky_description)/config/gaz_ros2_ctl_use_sim.yaml</parameters>
         </plugin>
-    </gazebo>
+    </gazebo> -->
+    <gazebo>
+  <plugin filename="gz_ros2_control-system" name="gz_ros2_control::GazeboSimROS2ControlPlugin">
+    <parameters>$(find rocky_controller)/config/my_controllers.yaml</parameters>
+    <parameters>$(find rocky_description)/config/gaz_ros2_ctl_use_sim.yaml</parameters>
+  </plugin>
+</gazebo>
 </robot>

Commit message: before tryinf drive on heading

File: rocky/src/rocky_description/urdf/camera.xacro (robot description, xacro)
@@ -1,11 +1,12 @@
 <?xml version="1.0"?>
-<robot xmlns:xacro="http://www.ros.org/wiki/xacro" >
+<robot xmlns:xacro="http://www.ros.org/wiki/xacro">
     <joint name="camera_joint" type="fixed">
         <parent link="chassis"/>
         <child link="camera_link"/>
-        <origin xyz="0.305 0 0.08" rpy="0 0 0"/> <!-- Changed from -1.5708 to 0 -->
+        <origin xyz="0.335 0 0.06" rpy="0 0 0"/>
     </joint>
     <link name="camera_link">
         <visual>
+            <origin xyz="0 0 0" rpy="0 0 0"/>
             <geometry>
                 <box size="0.010 0.03 0.03"/>
@@ -13,4 +14,10 @@
             <material name="rocky_red"/>
         </visual>
+        <!-- <collision>
+            <origin xyz="0 0 0" rpy="0 0 0"/>
+            <geometry>
+                <box size="0.010 0.03 0.03"/>
+            </geometry>
+        </collision> -->
     </link>
     <joint name="camera_optical_joint" type="fixed">
@@ -21,28 +28,27 @@
     <link name="camera_link_optical"></link>
     <gazebo reference="camera_link">
-        <material>Gazebo/Red</material>
-        <sensor name="camera" type="camera">
-            <pose> 0 0 0 0 0 0 </pose>
-            <visualize>true</visualize>
-            <update_rate>10</update_rate>
-            <camera>
-                <horizontal_fov>1.089</horizontal_fov>
+        <sensor name="camera" type="rgbd_camera">
+            <always_on>true</always_on>
+            <update_rate>30</update_rate>
+            <topic>camera</topic>
+            <gz_frame_id>camera_link</gz_frame_id>
+            <camera name="camera">
+                <horizontal_fov>0.96</horizontal_fov>
                 <image>
-                    <format>R8G8B8</format>
                     <width>640</width>
                     <height>480</height>
+                    <format>R8G8B8</format>
                 </image>
                 <clip>
-                    <near>0.05</near>
-                    <far>8.0</far>
+                    <near>0.1</near>
+                    <far>10.0</far>
                 </clip>
+                <depth_camera>
+                    <clip>
+                        <near>0.1</near>
+                        <far>10.0</far>
+                    </clip>
+                </depth_camera>
             </camera>
-            <!-- <plugin name="camera_controller" filename="libgazebo_ros_camera.so">
-                <frame_name>camera_link_optical</frame_name>
-            </plugin> -->
-            <!-- <plugin filename="gz-sim-sensors-system" name="gz::sim::systems::Sensors">
-            <render_engine>ogre2</render_engine>
-            </plugin> -->
-<!-- topic is set via <topic> tag on the <sensor> element -->
         </sensor>
     </gazebo>

File: rocky/src/rocky_description/urdf/depth_camera.xacro (robot description, xacro)
@@ -24,6 +24,8 @@
         <sensor name="camera" type="depth">
             <pose> 0 0 0 0 0 0 </pose>
+            <always_on>1</always_on>
             <visualize>true</visualize>
             <update_rate>10</update_rate>
+            <topic>camera</topic>
             <camera>
                 <horizontal_fov>2</horizontal_fov>
@@ -43,7 +45,7 @@
                 <max_depth>8.0</max_depth>
              </plugin> -->
-             <!-- <plugin filename="gz-sim-sensors-system" name="gz::sim::systems::Sensors">
-            <render_engine>ogre2</render_engine>
-            <min_depth>0.1</min_depth>
+             <!-- <plugin filename="gz-sim-sensors-system" name="gz::sim::systems::Sensors"> -->
+            <!-- <render_engine>ogre2</render_engine> -->
+            <!-- <min_depth>0.1</min_depth>
                 <max_depth>8.0</max_depth>
             </plugin> -->

File: rocky/src/rocky_description/urdf/rocky.urdf.xacro (robot description, xacro)
@@ -11,6 +11,6 @@
     </xacro:unless>
     <xacro:include filename="lidar.xacro" />
-    <!-- <xacro:include filename="camera.xacro" /> -->
-    <xacro:include filename="depth_camera.xacro" />
+    <xacro:include filename="camera.xacro" />
+    <!-- <xacro:include filename="depth_camera.xacro" /> -->
     <xacro:include filename="imu.xacro" />
     <!-- <xacro:include filename="face.xacro" /> -->

File: rocky/src/rocky_description/urdf/rocky_core.xacro (robot description, xacro)
@@ -99,6 +99,6 @@
     <gazebo reference="left_wheel">
         <material>Gazebo/Blue</material>
-     <mu1>1.0</mu1>
-<mu2>1.0</mu2>
+     <mu1>0.5</mu1>
+<mu2>0.5</mu2>
     </gazebo>
     <!-- RIGHT WHEEL LINK -->
@@ -127,6 +127,6 @@
     <gazebo reference="right_wheel">
         <material>Gazebo/Blue</material>
-       <mu1>1.0</mu1>
-<mu2>1.0</mu2>
+       <mu1>0.5</mu1>
+<mu2>0.5</mu2>
     </gazebo>
     <!-- CASTER WHEEL LINK -->
@@ -145,5 +145,5 @@
         <collision>
             <geometry>
-                <sphere radius="${caster_wheel_radius}" value="0.015"/>
+                <sphere radius="${caster_wheel_radius}" />
             </geometry>
         </collision>

Commit message: integrated vision output

File: rocky/src/rocky_description/urdf/camera.xacro (robot description, xacro)
@@ -4,5 +4,5 @@
         <parent link="chassis"/>
         <child link="camera_link"/>
-        <origin xyz="0.335 0 0.06" rpy="0 0 0"/>
+        <origin xyz="0.335 -0.001 0.09" rpy="0 0 0"/>
     </joint>
     <link name="camera_link">
@@ -41,5 +41,5 @@
                 </image>
                 <clip>
-                    <near>0.1</near>
+                    <near>0.01</near>
                     <far>10.0</far>
                 </clip>

File: rocky/src/rocky_description/urdf/rocky_core.xacro (robot description, xacro)
@@ -16,4 +16,5 @@
     <xacro:property name="caster_wheel_offset_x" value="0.075"/>
     <xacro:property name="caster_wheel_offset_z" value="${wheel_offset_z - wheel_radius + caster_wheel_radius}"/>
+    <xacro:property name="mast_radius" value="0.015"/> <xacro:property name="mast_height" value="0.028"/>  ```
     <material name="rocky_white">
         <color rgba="1 1 1 1" />
