Commit message: Remove mast_radius property
Removed mast_radius property from rocky_core.xacro.

File: rocky/src/rocky_description/urdf/rocky_core.xacro (robot description, xacro)
@@ -16,5 +16,4 @@
     <xacro:property name="caster_wheel_offset_x" value="0.075"/>
     <xacro:property name="caster_wheel_offset_z" value="${wheel_offset_z - wheel_radius + caster_wheel_radius}"/>
-    <xacro:property name="mast_radius" value="0.015"/> <xacro:property name="mast_height" value="0.028"/>  ```
     <material name="rocky_white">
         <color rgba="1 1 1 1" />

Commit message: Change collision geometry from sphere to cylinder

File: rocky/src/rocky_description/urdf/rocky_core.xacro (robot description, xacro)
@@ -118,5 +118,5 @@
         <collision>
             <geometry>
-                <sphere radius="${wheel_radius}" length="${wheel_thickness}"/>
+               <cylinder radius="${wheel_radius}" length="${wheel_thickness}"/>
             </geometry>
         </collision>
